Commit message: wsg_50_simulation: update urdf for simulation

File: wsg_50_simulation/urdf/wsg_50.urdf.xacro (robot description, xacro)
@@ -15,5 +15,5 @@
  </joint>
 <!-- BASE LINK -->
- <link name="${name}_base_link">
+  <link name="${name}_base_link">
       <inertial>
           <mass value="0.25" />
@@ -63,9 +63,13 @@
      <limit effort="100" velocity="100"/>
   </joint>
-  <transmission name="${name}_base_trans_left" type="pr2_mechanism_model/SimpleTransmission">
-     <actuator name="${name}_base_motor_left" />
-     <joint name="${name}_base_joint_gripper_left" />
-     <mechanicalReduction>1</mechanicalReduction>
-     <motorTorqueConstant>1</motorTorqueConstant>
+  <transmission name="${name}_base_trans_left">
+     <type>pr2_mechanism_model/SimpleTransmission</type>
+     <actuator name="${name}_base_motor_left">
+       <mechanicalReduction>1</mechanicalReduction>
+       <motorTorqueConstant>1</motorTorqueConstant>
+     </actuator>
+     <joint name="${name}_finger_left_joint" >
+        <hardwareInterface>hardware_interface/PositionJointInterface</hardwareInterface>
+     </joint>
   </transmission>
   <link name="${name}_gripper_left">
@@ -148,9 +152,13 @@
      <limit effort="100" velocity="100"/>
   </joint>
-  <transmission name="${name}_base_trans_right" type="pr2_mechanism_model/SimpleTransmission">
-     <actuator name="${name}_base_motor_right" />
-     <joint name="${name}_base_joint_gripper_right" />
-     <mechanicalReduction>1</mechanicalReduction>
-     <motorTorqueConstant>1</motorTorqueConstant>
+  <transmission name="${name}_base_trans_right">
+     <type>pr2_mechanism_model/SimpleTransmission</type>
+     <actuator name="${name}_base_motor_right" >
+       <mechanicalReduction>1</mechanicalReduction>
+       <motorTorqueConstant>1</motorTorqueConstant>
+     </actuator>
+     <joint name="${name}_finger_right_joint">
+        <hardwareInterface>hardware_interface/PositionJointInterface</hardwareInterface>
+     </joint>
   </transmission>
     <link name="${name}_gripper_right">

Commit message: Added updates to simulator for gripper so we can run it with traj controller

File: wsg_50_simulation/urdf/wsg_50.urdf.xacro (robot description, xacro)
@@ -22,5 +22,5 @@
                iyy="100.0" iyz="0.0"
                izz="1.0" /-->
-      	  <inertia  ixx="1.0" ixy="0.0"  ixz="0.0"  iyy="1.0"  iyz="0.0"  izz="1.0" />
+      	  <inertia  ixx="0.005" ixy="0.0"  ixz="0.0"  iyy="0.005"  iyz="0.0"  izz="0.005" />
       </inertial>
       <visual>
@@ -55,5 +55,5 @@
   <!-- GRIPPER LEFT -->
   <joint name="${name}_finger_left_joint" type="prismatic">
-     <limit lower="-0.055" upper="-0.0027" effort="1.0" velocity="1.0"/>
+     <limit lower="-0.055" upper="-0.0027" effort="1000.0" velocity="100.0"/>
      <origin xyz="0 0 0" rpy="0 0 0" />      <!--origin xyz="-0.0067 0 0.049" rpy="0 0 0" /-->
      <parent link="${name}_base_link"/>
@@ -61,14 +61,14 @@
      <dynamics friction="100" damping="100" />
      <axis xyz="1 0 0"/>
-     <limit effort="100" velocity="100"/>
+     <!--<limit effort="10000" velocity="100"/>-->
   </joint>
   <transmission name="${name}_base_trans_left">
-     <type>pr2_mechanism_model/SimpleTransmission</type>
+     <type>transmission_interface/SimpleTransmission</type>
      <actuator name="${name}_base_motor_left">
-       <mechanicalReduction>1</mechanicalReduction>
-       <motorTorqueConstant>1</motorTorqueConstant>
+       <mechanicalReduction>100</mechanicalReduction>
+       <motorTorqueConstant>0.01</motorTorqueConstant>
      </actuator>
      <joint name="${name}_finger_left_joint" >
-        <hardwareInterface>hardware_interface/PositionJointInterface</hardwareInterface>
+        <hardwareInterface>hardware_interface/EffortJointInterface</hardwareInterface>
      </joint>
   </transmission>
@@ -76,8 +76,8 @@
       <inertial>
           <mass value="0.1" />
-          <origin xyz="0 0 0" />
-      <inertia ixx="1.0" ixy="0.0" ixz="0.0"
-               iyy="1.0" iyz="0.0"
-               izz="1.0" />
+          <origin xyz="0 0 0.08" />
+      <inertia ixx="0.002" ixy="0.0" ixz="0.0"
+               iyy="0.001" iyz="0.0"
+               izz="0.001" />
       </inertial>
       <visual>
@@ -88,12 +88,12 @@
           </geometry>
           <material name="black">
-		<color rgba="0 0 0 0"/>
-      	  </material>
-      </visual>
-      <collision>
-          <origin xyz="0 0 0" rpy="0 0 0" />
-          <geometry>
-	     <!--box size="0.0175 0.03 0.024"/-->
-             <mesh filename="package://wsg_50_simulation/meshes/GUIDE_WSG50_110.stl" scale="0.001 0.001 0.001"/>
+		<color rgba="0 0 0 1.0"/>
+      	  </material>
+      </visual>
+      <collision>
+          <origin xyz="0 0 0" rpy="0 0 0" />
+          <geometry>
+	     <!--box size="0.0175 0.03 0.024"/-->
+            <mesh filename="package://wsg_50_simulation/meshes/GUIDE_WSG50_110.stl" scale="0.001 0.001 0.001"/>
          </geometry>
      </collision>
@@ -116,8 +116,8 @@
       <inertial>
           <mass value="0.1" />
-          <origin xyz="0 0 0" />
-      <inertia ixx="1.0" ixy="0.0" ixz="0.0"
-               iyy="1.0" iyz="0.0"
-               izz="1.0" />
+          <origin xyz="0 0 0.12" />
+      <inertia ixx="0.002" ixy="0.0" ixz="0.0"
+               iyy="0.001" iyz="0.0"
+               izz="0.001" />
       </inertial>
       <visual>
@@ -144,5 +144,5 @@
   <!-- GRIPPER RIGHT -->
   <joint name="${name}_finger_right_joint" type="prismatic">
-     <limit lower="0.0027" upper="0.055" effort="1.0" velocity="1.0"/>
+     <limit lower="0.0027" upper="0.055" effort="1000.0" velocity="100.0"/>
      <origin xyz="0 0 0" rpy="0 0 3.14159" />
      <parent link="${name}_base_link"/>
@@ -150,14 +150,14 @@
      <axis xyz="-1 0 0"/>
      <dynamics friction="100" damping="100" />
-     <limit effort="100" velocity="100"/>
+     <!--<limit effort="10000" velocity="100"/>-->
   </joint>
   <transmission name="${name}_base_trans_right">
-     <type>pr2_mechanism_model/SimpleTransmission</type>
+     <type>transmission_interface/SimpleTransmission</type>
      <actuator name="${name}_base_motor_right" >
-       <mechanicalReduction>1</mechanicalReduction>
-       <motorTorqueConstant>1</motorTorqueConstant>
+       <mechanicalReduction>100</mechanicalReduction>
+       <motorTorqueConstant>0.01</motorTorqueConstant>
      </actuator>
      <joint name="${name}_finger_right_joint">
-        <hardwareInterface>hardware_interface/PositionJointInterface</hardwareInterface>
+        <hardwareInterface>hardware_interface/EffortJointInterface</hardwareInterface>
      </joint>
   </transmission>
@@ -165,8 +165,8 @@
       <inertial>
           <mass value="0.1" />
-          <origin xyz="0 0 0" />
-      <inertia ixx="1.0" ixy="0.0" ixz="0.0"
-               iyy="1.0" iyz="0.0"
-               izz="1.0" />
+          <origin xyz="0 0 0.08" />
+      <inertia ixx="0.002" ixy="0.0" ixz="0.0"
+               iyy="0.001" iyz="0.0"
+               izz="0.001" />
       </inertial>
       <visual>
@@ -177,5 +177,5 @@
           </geometry>
           <material name="black">
-		<color rgba="0 0 0 0"/>
+		<color rgba="0 0 0 1.0"/>
       	  </material>
       </visual>
@@ -190,6 +190,12 @@
   </link>
   <gazebo reference="gripper_right">
-    <material>Gazebo/White</material>
-    <turnGravityOff>false</turnGravityOff>
+    <material>Gazebo/Black</material>
+    <turnGravityOff>false</turnGravityOff>
+    <kp>1000000.0</kp>
+    <kd>100.0</kd>
+    <mu1>30.0</mu1>
+    <mu2>30.0</mu2>
+    <maxVel>1.0</maxVel>
+    <minDepth>0.001</minDepth>
   </gazebo>
   <!-- RIGHT FINGER -->
@@ -205,16 +211,16 @@
       <inertial>
           <mass value="0.1" />
-          <origin xyz="0 0 0" />
-      <inertia ixx="1.0" ixy="0.0" ixz="0.0"
-               iyy="1.0" iyz="0.0"
-               izz="1.0" />
-      </inertial>
-      <visual>
-          <origin xyz="0.0 0 0" rpy="0 0 0" />
-          <geometry>
-             <mesh filename="package://wsg_50_simulation/meshes/WSG-FMF.stl" scale="0.001 0.001 0.001"/>
-          </geometry>
-          <material name="black">
-		<color rgba="0 0 0 0"/>
+          <origin xyz="0 0 0.12" />
+      <inertia ixx="0.002" ixy="0.0" ixz="0.0"
+               iyy="0.0" iyz="0.0"
+               izz="0.0" />
+      </inertial>
+      <visual>
+          <origin xyz="0.0 0 0" rpy="0 0 0" />
+          <geometry>
+             <mesh filename="package://wsg_50_simulation/meshes/WSG-FMF.stl" scale="0.001 0.001 0.001"/>
+          </geometry>
+          <material name="black">
+		<color rgba="0 0 0 1.0"/>
       	  </material>
       </visual>
@@ -228,6 +234,12 @@
   </link>
   <gazebo reference="${name}_finger_right">
-    <material>Gazebo/White</material>
-    <turnGravityOff>false</turnGravityOff>
+    <material>Gazebo/Black</material>
+    <turnGravityOff>false</turnGravityOff>
+    <kp>1000000.0</kp>
+    <kd>100.0</kd>
+    <mu1>30.0</mu1>
+    <mu2>30.0</mu2>
+    <maxVel>1.0</maxVel>
+    <minDepth>0.001</minDepth>
   </gazebo>
 </xacro:macro>

Commit message: Reduced friction to allow the gripper to reach its goal

File: wsg_50_simulation/urdf/wsg_50.urdf.xacro (robot description, xacro)
@@ -59,5 +59,5 @@
      <parent link="${name}_base_link"/>
      <child link="${name}_gripper_left" />
-     <dynamics friction="100" damping="100" />
+     <dynamics friction="20" damping="100" />
      <axis xyz="1 0 0"/>
      <!--<limit effort="10000" velocity="100"/>-->
@@ -149,5 +149,5 @@
      <child link="${name}_gripper_right" />
      <axis xyz="-1 0 0"/>
-     <dynamics friction="100" damping="100" />
+     <dynamics friction="20" damping="100" />
      <!--<limit effort="10000" velocity="100"/>-->
   </joint>
